File: 3.3v_BuckBoost.kicad_sch (KiCad schematic)
At the start: 7 parts, among them U801 TPS63031DSK

Commit message: "V1.0 final design"
Parts:
- L801: footprint Inductor_SMD_Wurth:L_Wurth_WE-LQSH-4020 -> Inductor_SMD:L_KOHERelec_MDA7030
Changed lines of the file:
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@@
 			)
 		)
-		(property "Footprint" "Inductor_SMD_Wurth:L_Wurth_WE-LQSH-4020"
+		(property "Footprint" "Inductor_SMD:L_KOHERelec_MDA7030"
 			(at 127 99.06 0)
 			(effects
