File: 5V_Boost_Converter.kicad_sch (KiCad schematic)
At the start: 8 parts, among them U901 TPS61023DRLR

Commit message: "V1.0 final design"
Parts:
- U901: footprint TPS61023DRLR:SOT563-ORI -> govi_v3_sensor_footprints_kicad:SOT563-ORI
Changed lines of the file:
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@@
 			)
 		)
-		(property "Footprint" "TPS61023DRLR:SOT563-ORI"
+		(property "Footprint" "govi_v3_sensor_footprints_kicad:SOT563-ORI"
 			(at 144.78 97.79 0)
 			(effects
