File: AC_power_module.kicad_sch (KiCad schematic)
At the start: 7 parts, among them J401 7.62mm 2-Pin Screw Terminal

Commit message: "V1.0 final design"
Parts:
- J401: footprint govi_v3_sensor_footprints_kicad:P=7.62mm Barrier Terminal Blocks azend -> Connector_Phoenix_MC_HighVoltage:PhoenixContact_MCV_1,5_2-G-5.08_1x02_P5.08mm_Vertical
Changed lines of the file:
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@@
 			)
 		)
-		(property "Footprint" "govi_v3_sensor_footprints_kicad:P=7.62mm Barrier Terminal Blocks azend"
+		(property "Footprint" "Connector_Phoenix_MC_HighVoltage:PhoenixContact_MCV_1,5_2-G-5.08_1x02_P5.08mm_Vertical"
 			(at 96.52 99.06 0)
 			(effects
