File: Battery_Module.kicad_sch (KiCad schematic)
At the start: 10 parts, among them Q701 FS8205A, U701 DW01A

Commit message: "V1.0 final design"
Parts:
- removed BT701: Battery_Cell, govi_v3_sensor_footprints_kicad:BAT_1042P, symbol Device:Battery_Cell
- added J601: Conn_01x02, Connector_Phoenix_MC_HighVoltage:PhoenixContact_MCV_1,5_2-G-5.08_1x02_P5.08mm_Vertical, symbol Connector_Generic:Conn_01x02
Connections:
- net BAT+: now also J601.1 (Pin_1)
- net BAT-: no longer TP701.1
- net at C701.2, Q701.2, Q701.3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: now also TP701.1, J601.2 (Pin_2)
Other:
- moved on the sheet: TP701
Changed lines of the file:
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@@
-	)
-	(junction
-		(at 73.66 113.03)
-		(diameter 0)
-		(color 0 0 0 0)
 	)
 	(junction
@@
 	)
 	(junction
-		(at 162.56 85.09)
-		(diameter 0)
-		(color 0 0 0 0)
-	)
-	(junction
 		(at 78.74 125.73)
 		(diameter 0)
@@
 	)
 	(junction
+		(at 123.19 113.03)
+		(diameter 0)
+		(color 0 0 0 0)
+	)
+	(junction
 		(at 231.14 92.71)
 		(diameter 0)
@@
 	(wire
 		(pts
-			(xy 107.95 113.03) (xy 156.21 113.03)
-		)
-		(stroke
-			(width 0)
-			(type default)
-		)
-	)
-	(wire
-		(pts
-			(xy 156.21 85.09) (xy 156.21 95.25)
+			(xy 107.95 113.03) (xy 123.19 113.03)
+		)
+		(stroke
+			(width 0)
+			(type default)
+		)
+	)
+	(wire
+		(pts
+			(xy 123.19 113.03) (xy 156.21 113.03)
 		)
 		(stroke
@@
 	(wire
 		(pts
-			(xy 162.56 85.09) (xy 177.8 85.09)
-		)
-		(stroke
-			(width 0)
-			(type default)
-		)
-	)
-	(wire
-		(pts
 			(xy 144.78 85.09) (xy 144.78 95.25)
 		)
@@
 	(wire
 		(pts
-			(xy 156.21 85.09) (xy 162.56 85.09)
+			(xy 156.21 85.09) (xy 177.8 85.09)
 		)
 		(stroke
@@
 	(wire
 		(pts
+			(xy 156.21 97.79) (xy 158.75 97.79)
+		)
+		(stroke
+			(width 0)
+			(type default)
+		)
+	)
+	(wire
+		(pts
 			(xy 95.25 95.25) (xy 95.25 100.33)
 		)
@@
 	(wire
 		(pts
-			(xy 73.66 107.95) (xy 73.66 113.03)
-		)
-		(stroke
-			(width 0)
-			(type default)
-		)
-	)
-	(wire
-		(pts
 			(xy 95.25 100.33) (xy 97.79 100.33)
 		)
@@
 	(wire
 		(pts
+			(xy 156.21 85.09) (xy 156.21 97.79)
+		)
+		(stroke
+			(width 0)
+			(type default)
+		)
+	)
+	(wire
+		(pts
 			(xy 107.95 90.17) (xy 102.87 90.17)
 		)
@@
 	(wire
 		(pts
-			(xy 73.66 113.03) (xy 80.01 113.03)
+			(xy 158.75 100.33) (xy 156.21 100.33)
+		)
+		(stroke
+			(width 0)
+			(type default)
+		)
+	)
+	(wire
+		(pts
+			(xy 63.5 113.03) (xy 80.01 113.03)
 		)
 		(stroke
@@
 	(wire
 		(pts
-			(xy 63.5 113.03) (xy 73.66 113.03)
-		)
-		(stroke
-			(width 0)
-			(type default)
-		)
-	)
-	(wire
-		(pts
-			(xy 162.56 80.01) (xy 162.56 85.09)
+			(xy 123.19 107.95) (xy 123.19 113.03)
 		)
 		(stroke
@@
 	(wire
 		(pts
-			(xy 156.21 102.87) (xy 156.21 113.03)
+			(xy 156.21 100.33) (xy 156.21 113.03)
 		)
 		(stroke
@@
 	)
 	(symbol
-		(lib_id "power:PWR_FLAG")
-		(at 162.56 80.01 0)
-		(unit 1)
-		(exclude_from_sim no)
-		(in_bom yes)
-		(on_board yes)
-		(dnp no)
-		(fields_autoplaced yes)
-		(property "Reference" "#FLG0703"
-			(at 162.56 78.105 0)
-			(effects
-				(font
-					(size 1.27 1.27)
-				)
-				(hide yes)
-			)
-		)
-		(property "Value" "PWR_FLAG"
-			(at 162.56 74.93 0)
-			(effects
-				(font
-					(size 1.27 1.27)
-				)
-			)
-		)
-		(property "Footprint" ""
-			(at 162.56 80.01 0)
-			(effects
-				(font
-					(size 1.27 1.27)
-				)
-				(hide yes)
-			)
-		)
-		(property "Datasheet" "~"
-			(at 162.56 80.01 0)
-			(effects
-				(font
-					(size 1.27 1.27)
-				)
-				(hide yes)
-			)
-		)
-		(property "Description" "Special symbol for telling ERC where power comes from"
-			(at 162.56 80.01 0)
-			(effects
-				(font
-					(size 1.27 1.27)
-				)
-				(hide yes)
-			)
-		)
-		(pin "1"
-		)
-		(instances
-			(project "govi_v3_SHT41_sensor_kicad"
-				(path "/ba95ddf4-72c6-4eeb-9c09-ae7c8e5af670/625f4f9c-da9a-4f02-8306-7d03107693c0"
-					(reference "#FLG0703")
-					(unit 1)
-				)
-			)
-		)
-	)
-	(symbol
 		(lib_id "Device:R")
 		(at 220.98 92.71 90)
@@
 	)
 	(symbol
+		(lib_id "Connector_Generic:Conn_01x02")
+		(at 163.83 97.79 0)
+		(unit 1)
+		(exclude_from_sim no)
+		(in_bom yes)
+		(on_board yes)
+		(dnp no)
+		(fields_autoplaced yes)
+		(property "Reference" "J601"
+			(at 166.37 97.7899 0)
+			(effects
+				(font
+					(size 1.27 1.27)
+				)
+				(justify left)
+			)
+		)
+		(property "Value" "Conn_01x02"
+			(at 166.37 100.3299 0)
+			(effects
+				(font
+					(size 1.27 1.27)
+				)
+				(justify left)
+			)
+		)
+		(property "Footprint" "Connector_Phoenix_MC_HighVoltage:PhoenixContact_MCV_1,5_2-G-5.08_1x02_P5.08mm_Vertical"
+			(at 163.83 97.79 0)
+			(effects
+				(font
+					(size 1.27 1.27)
+				)
+				(hide yes)
+			)
+		)
+		(property "Datasheet" "~"
+			(at 163.83 97.79 0)
+			(effects
+				(font
+					(size 1.27 1.27)
+				)
+				(hide yes)
+			)
+		)
+		(property "Description" "Generic connector, single row, 01x02, script generated (kicad-library-utils/schlib/autogen/connector/)"
+			(at 163.83 97.79 0)
+			(effects
+				(font
+					(size 1.27 1.27)
+				)
+				(hide yes)
+			)
+		)
+		(pin "1"
+		)
+		(pin "2"
+		)
+		(instances
+			(project ""
+				(path "/ba95ddf4-72c6-4eeb-9c09-ae7c8e5af670/625f4f9c-da9a-4f02-8306-7d03107693c0"
+					(reference "J601")
+					(unit 1)
+				)
+			)
+		)
+	)
+	(symbol
 		(lib_id "Device:C")
 		(at 144.78 99.06 0)
@@
 	(symbol
 		(lib_id "Connector:TestPoint")
-		(at 73.66 107.95 0)
+		(at 123.19 107.95 0)
 		(unit 1)
 		(exclude_from_sim no)
@@
 		(fields_autoplaced yes)
 		(property "Reference" "TP701"
-			(at 76.2 103.3779 0)
+			(at 125.73 103.3779 0)
 			(effects
 				(font
@@
 		)
 		(property "Value" "BAT-"
-			(at 76.2 105.9179 0)
+			(at 125.73 105.9179 0)
 			(effects
 				(font
@@
 		)
 		(property "Footprint" "TestPoint:TestPoint_Pad_D1.0mm"
-			(at 78.74 107.95 0)
+			(at 128.27 107.95 0)
 			(effects
 				(font
@@
 		)
 		(property "Datasheet" "~"
-			(at 78.74 107.95 0)
+			(at 128.27 107.95 0)
 			(effects
 				(font
@@
 		)
 		(property "Description" "test point"
-			(at 73.66 107.95 0)
+			(at 123.19 107.95 0)
 			(effects
 				(font
@@
 		)
 		(instances
-			(project ""
+			(project "govi_v3_Actuator_node_kicad"
 				(path "/ba95ddf4-72c6-4eeb-9c09-ae7c8e5af670/625f4f9c-da9a-4f02-8306-7d03107693c0"
 					(reference "TP701")
 					(unit 1)
 				)
-			)
-		)
-	)
-	(symbol
-		(lib_id "Device:Battery_Cell")
-		(at 156.21 100.33 0)
-		(unit 1)
-		(exclude_from_sim no)
-		(in_bom yes)
-		(on_board yes)
-		(dnp no)
-		(fields_autoplaced yes)
-		(property "Reference" "BT701"
-			(at 160.02 97.2184 0)
-			(effects
-				(font
-					(size 1.27 1.27)
-				)
-				(justify left)
-			)
-		)
-		(property "Value" "Battery_Cell"
-			(at 160.02 99.7584 0)
-			(effects
-				(font
-					(size 1.27 1.27)
-				)
-				(justify left)
-			)
-		)
-		(property "Footprint" "govi_v3_sensor_footprints_kicad:BAT_1042P"
-			(at 156.21 98.806 90)
-			(effects
-				(font
-					(size 1.27 1.27)
-				)
-				(hide yes)
-			)
-		)
-		(property "Datasheet" "~"
-			(at 156.21 98.806 90)
-			(effects
-				(font
-					(size 1.27 1.27)
-				)
-				(hide yes)
-			)
-		)
-		(property "Description" "Single-cell battery"
-			(at 156.21 100.33 0)
-			(effects
-				(font
-					(size 1.27 1.27)
-				)
-				(hide yes)
-			)
-		)
-		(pin "1"
-		)
-		(pin "2"
-		)
-		(instances
-			(project "govi_v3_SHT41_sensor_kicad"
-				(path "/ba95ddf4-72c6-4eeb-9c09-ae7c8e5af670/625f4f9c-da9a-4f02-8306-7d03107693c0"
-					(reference "BT701")
-					(unit 1)
-				)
