File: MCU.kicad_sch (KiCad schematic)
At the start: 22 parts, among them J201 Conn_01x03, J203 Conn_01x04, SW201 SW_Push, U201 STM32F103C6Tx, Y201 8 MHz

Commit message: "V1.0 final design"
Parts:
- removed JP201: SolderJumper_2_Open, Jumper:SolderJumper-2_P1.3mm_Open_RoundedPad1.0x1.5mm, symbol Jumper:SolderJumper_2_Open
Connections:
- net OUT_0: now also U201.28 (PB15); no longer U201.27 (PB14)
- net OUT_1: now also U201.27 (PB14); no longer U201.28 (PB15)
- net IN_2: now reaches U201.32 (PA11)
- net IN_3: now reaches U201.33 (PA12)
- no-connect marks 18 -> 16
Other:
- moved on the sheet: FB201, J201
