File: Output_driver.kicad_sch (KiCad schematic)
At the start: 12 parts, among them J1101 5.08mm 2P Screw Plug-in Termi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, J1102 5.08mm 2P Screw Plug-in Termi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, Q1101 BC817-40, Q1102 BC817-40, U1101 G3MB-202P, U1102 G3MB-202P

Commit message: "V1.0 final design"
Parts:
- removed J1101, J1102: 5.08mm 2P Screw Plug-in Terminal, Connector_Phoenix_MSTB:PhoenixContact_MSTBA_2,5_2-G-5,08_1x02_P5.08mm_Horizontal, symbol Connector_Generic:Conn_01x02
- removed Q1101, Q1102: BC817-40, Package_TO_SOT_SMD:SOT-23, symbol Device:Q_NPN
- added J1001: Conn_01x04, Connector_Phoenix_MC_HighVoltage:PhoenixContact_MCV_1,5_4-G-5.08_1x04_P5.08mm_Vertical, symbol Connector_Generic:Conn_01x04
- added Q1002, Q1101: BC817-40, Package_TO_SOT_SMD:SOT-23, symbol Transistor_BJT:BC817
- C1101, C1102: value 0.1MFD -> 0.1uF
- U1101, U1102: footprint OptoDevice:Finder_34.81 -> govi_v3_sensor_footprints_kicad:G3MB202PLDC5
Connections:
- net GND: now also Q1002.2 (E), Q1101.2 (E)
- net OUT1_11: now reaches U1102.11
- net OUT1_11: now also J1001.4 (Pin_4)
- net OUT1_14: now reaches U1102.14
- net OUT1_14: now also J1001.3 (Pin_3)
- net at R1102.2: now also Q1101.1 (B)
- net at C1101.2, U1101.A2: now also Q1101.3 (C)
- net OUT0_11: now reaches U1101.11
- net OUT0_11: now also J1001.2 (Pin_2)
- net OUT0_14: now reaches U1101.14
- net OUT0_14: now also J1001.1 (Pin_1)
- net at R1103.2: now also Q1002.1 (B)
- net at C1102.2, U1102.A2: now also Q1002.3 (C)
