File: govi_v3_Actuator_node_kicad.kicad_pcb (KiCad board)
At the start: 2 copper layers, 74 x 108 mm, 106 parts, among them J1001 5.08mm 2P Screw Plug-in Termi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, J1002 5.08mm 2P Screw Plug-in Termi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, J1101 5.08mm 2P Screw Plug-in Termi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, J1102 5.08mm 2P Screw Plug-in Termi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, J201 Conn_01x03, J203 Conn_01x04, J401 7.62mm 2-Pin Screw Terminal, J501 7.62mm 2-Pin Screw Terminal, Q1101 BC817-40, Q1102 BC817-40, Q501 Q_PMOS_Depletion, Q701 FS8205A, SW201 SW_Push, U1001 PC817, U1002 PC817, U1101 G3MB-202P, U1102 G3MB-202P, U201 STM32F103C6Tx, U301 Ra-02, U501 CN3791, U601 TP4056-42-ESOP8-AMS, U701 DW01A, U801 TPS63031DSK, U901 TPS61023DRLR, Y201 8 MHz

Commit message: "V1.0 final design"
Parts:
- removed BT701: Battery_Cell, govi_v3_sensor_footprints_kicad:BAT_1042P
- removed C501, C506: 10uF, Capacitor_SMD:C_0603_1608Metric_Pad1.08x0.95mm_HandSolder
- removed C502: 47nF, Capacitor_SMD:C_0603_1608Metric_Pad1.08x0.95mm_HandSolder
- removed C503: 220uF 35V, Capacitor_SMD:CP_Elec_6.3x7.7
- removed C504: 0.1uF, Capacitor_SMD:C_0603_1608Metric_Pad1.08x0.95mm_HandSolder
- removed C505: 0.22µF, Capacitor_SMD:C_0603_1608Metric_Pad1.08x0.95mm_HandSolder
- removed C507: 10uF 20V, Capacitor_Tantalum_SMD:CP_EIA-3216-18_Kemet-A_HandSolder
- removed D502, D503, D601: SS54, Diode_SMD:D_SMA
- removed the G*** at (27.7, 63.9)
- removed the G*** at (-14.4, 60.2)
- removed J1002, J1101, J1102: 5.08mm 2P Screw Plug-in Terminal, Connector_Phoenix_MSTB:PhoenixContact_MSTBA_2,5_2-G-5,08_1x02_P5.08mm_Horizontal
- removed J501: 7.62mm 2-Pin Screw Terminal, govi_v3_sensor_footprints_kicad:P=7.62mm Barrier Terminal Blocks azend
- removed JP201: SolderJumper_2_Open, Jumper:SolderJumper-2_P1.3mm_Open_RoundedPad1.0x1.5mm
- removed L501: 82µH 12x12mm, Inductor_SMD:L_12x12mm_H4.5mm
- removed Q1102: BC817-40, Package_TO_SOT_SMD:SOT-23
- removed Q501: Q_PMOS_Depletion, Package_TO_SOT_SMD:TO-252-2
- removed R501: 120R, Resistor_SMD:R_0603_1608Metric_Pad0.98x0.95mm_HandSolder
- removed R502: 133K, Resistor_SMD:R_0603_1608Metric_Pad0.98x0.95mm_HandSolder
- removed R503: 10K, Resistor_SMD:R_0603_1608Metric_Pad0.98x0.95mm_HandSolder
- removed R504: R040 40mΩ, Resistor_SMD:R_2512_6332Metric_Pad1.40x3.35mm_HandSolder
- removed TP501: MPPT, TestPoint:TestPoint_Pad_D1.0mm
- removed U501: CN3791, Package_SO:SSOP-10_3.9x4.9mm_P1.00mm
- added C904: 0.1uF, Capacitor_SMD:C_0402_1005Metric_Pad0.74x0.62mm_HandSolder, B.Cu at (154.6, 103.1)
- added C905: 0.1uF, Capacitor_SMD:C_0402_1005Metric_Pad0.74x0.62mm_HandSolder, B.Cu at (146.5, 103.1)
- added G***: LOGO, govi_v3_sensor_footprints_kicad:logo, F.Cu at (151.8, 87.5)
- added G***: LOGO, govi_v3_sensor_footprints_kicad:govi-ai-logo-back, B.Cu at (131.3, 92.2)
- added J601: Conn_01x02, Connector_Phoenix_MC_HighVoltage:PhoenixContact_MCV_1,5_2-G-5.08_1x02_P5.08mm_Vertical, F.Cu at (163.6, 135.9)
- added J901: Conn_01x04, Connector_Phoenix_MC_HighVoltage:PhoenixContact_MCV_1,5_4-G-5.08_1x04_P5.08mm_Vertical, F.Cu at (153.6, 115.7)
- added Q1002: BC817-40, Package_TO_SOT_SMD:SOT-23, F.Cu at (170.7, 107.4)
- added R1007: 1K, Resistor_SMD:R_0603_1608Metric_Pad0.98x0.95mm_HandSolder, F.Cu at (139.7, 103.6)
- added R1008: 100K, Resistor_SMD:R_0402_1005Metric_Pad0.72x0.64mm_HandSolder, B.Cu at (146.5, 100.1)
- added R1009: 4.7K, Resistor_SMD:R_0402_1005Metric_Pad0.72x0.64mm_HandSolder, F.Cu at (139.7, 99.2)
- added R1010: 1K, Resistor_SMD:R_0603_1608Metric_Pad0.98x0.95mm_HandSolder, F.Cu at (147.9, 103.6)
- added R1011: 100K, Resistor_SMD:R_0402_1005Metric_Pad0.72x0.64mm_HandSolder, B.Cu at (154.6, 100.1)
- added R1012: 4.7K, Resistor_SMD:R_0402_1005Metric_Pad0.72x0.64mm_HandSolder, F.Cu at (147.9, 99.2)
- added U902: PC817, Package_DIP:DIP-4_W7.62mm, F.Cu at (150.3, 105.4)
- added U903: PC817, Package_DIP:DIP-4_W7.62mm, F.Cu at (142.1, 105.4)
- C1001: value 0.1MFD -> 0.1uF
- C1002, C1101, C1102: value 0.1MFD -> 0.1uF; moved to B.Cu
- C701, C702, C901, C902, C903, L901, Q701, R1001, R1002, R701, R702, R901, R902, U1001, U701: moved to F.Cu
- J1001: value 5.08mm 2P Screw Plug-in Terminal -> Conn_01x04; footprint Connector_Phoenix_MSTB:PhoenixContact_MSTBA_2,5_2-G-5,08_1x02_P5.08mm_Horizontal -> Connector_Phoenix_MC_HighVoltage:PhoenixContact_MCV_1,5_4-G-5.08_1x04_P5.08mm_Vertical
- J401: footprint govi_v3_sensor_footprints_kicad:P=7.62mm Barrier Terminal Blocks azend -> Connector_Phoenix_MC_HighVoltage:PhoenixContact_MCV_1,5_2-G-5.08_1x02_P5.08mm_Vertical
- L801: footprint Inductor_SMD_Wurth:L_Wurth_WE-LQSH-4020 -> Inductor_SMD:L_KOHERelec_MDA7030
- R1003, R1005, R1101, R1104: moved to B.Cu
- U1101, U1102: footprint OptoDevice:Finder_34.81 -> govi_v3_sensor_footprints_kicad:G3MB202PLDC5
- U901: footprint govi_v3_sensor_footprint_kicad:SOT563-ORI -> govi_v3_sensor_footprints_kicad:SOT563-ORI; moved to F.Cu
- moved R1104 239.3 mm to (167.0, 96.6), turned to -90 degrees
- moved U1102 238.2 mm to (170.2, 81.8), turned to 90 degrees
- moved R1103 233.4 mm to (166.8, 107.4), turned to 90 degrees
- moved R1101 230.7 mm to (158.7, 96.5), turned to -90 degrees
- moved C1102 230.2 mm to (167.0, 101.6), turned to -90 degrees
- moved U1101 229.3 mm to (161.7, 81.7), turned to 90 degrees
- moved R1102 224.7 mm to (158.3, 107.4), turned to 90 degrees
- moved C1101 221.8 mm to (158.7, 101.5), turned to -90 degrees
- moved Q1101 204.1 mm to (162.2, 107.4)
- moved U1002 194.7 mm to (158.7, 120.7), turned to -90 degrees
- moved R1003 186.5 mm to (162.5, 126.0), turned to -90 degrees
- moved U1001 186.4 mm to (166.8, 120.7)
- moved R1002 186.0 mm to (169.3, 126.9)
- moved R1004 185.9 mm to (161.1, 122.5), turned to 90 degrees
- moved R1006 184.7 mm to (161.1, 126.9), turned to 90 degrees
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Connections:
- net Net-(J1002-Pin_1) renamed /Input_driver/IN1
- C1001 pad 2: Net-(J1001-Pin_1) -> /Input_driver/IN0
- C1101 pad 2: Net-(C1101-Pad2) -> Net-(Q1101-C)
- C701 pad 2: Net-(BT701--) -> Net-(J601-Pin_2)
- J1001 pad 1: Net-(J1001-Pin_1) -> /Output_driver/OUT0_14
- J1001 pad 2: GND -> /Output_driver/OUT0_11
- Q1101 pad 1: (no net) -> Net-(Q1101-B)
- Q1101 pad 2: (no net) -> GND
- Q1101 pad 3: (no net) -> Net-(Q1101-C)
- Q701 pad 2: Net-(BT701--) -> Net-(J601-Pin_2)
- Q701 pad 3: Net-(BT701--) -> Net-(J601-Pin_2)
- R1102 pad 2: Net-(Q1101-PadB) -> Net-(Q1101-B)
- TP601 pad 1: Net-(D601-A) -> /Battery_Module/BAT(+)
- TP701 pad 1: GND -> Net-(J601-Pin_2)
- U1001 pad 2: Net-(J1001-Pin_1) -> /Input_driver/IN0
- U1101 pad 11: Net-(J1101-Pin_1) -> /Output_driver/OUT0_11
- U1101 pad 14: Net-(J1101-Pin_2) -> /Output_driver/OUT0_14
- U1101 pad A2: Net-(C1101-Pad2) -> Net-(Q1101-C)
- U1102 pad 11: Net-(J1102-Pin_1) -> /Output_driver/OUT1_11
- U1102 pad 14: Net-(J1102-Pin_2) -> /Output_driver/OUT1_14
- U201 pad 27: /MCU/OUT_0 -> /MCU/OUT_1
- U201 pad 28: /MCU/OUT_1 -> /MCU/OUT_0
- U201 pad 32: unconnected-(U201-PA11-Pad32) -> /Input_driver/INPUT2
- U201 pad 33: unconnected-(U201-PA12-Pad33) -> /Input_driver/INPUT3
- U601 pad 5: Net-(D601-A) -> /Battery_Module/BAT(+)
- U701 pad 6: Net-(BT701--) -> Net-(J601-Pin_2)
Routing:
- net Net-(BT701--): track 109.8 -> 0.00 mm, vias 1 -> 0
- net Net-(D503-A): track 64.4 -> 0.00 mm, vias 1 -> 0
- net +5VD: track 44.2 -> 103.5 mm, vias 0 -> 2
- net /Battery_Module/BAT(+): track 85.8 -> 142.7 mm, vias 3 -> 0
- net /Input_driver/INPUT3: track 0.00 -> 50.4 mm, vias 0 -> 1
- net /Input_driver/INPUT2: track 0.00 -> 39.1 mm, vias 0 -> 1
- net +12V: track 38.5 -> 0.00 mm
- net Net-(J601-Pin_2): track 0.00 -> 37.3 mm
- net /MCU/OUT_1: track 0.00 -> 36.5 mm
- net /Input_driver/INPUT0: track 0.00 -> 36.0 mm
- net +3V3: track 134.2 -> 169.5 mm, vias 8 -> 5
- net /Input_driver/INPUT1: track 0.00 -> 28.3 mm
- net /MCU/OUT_0: track 0.00 -> 27.7 mm
- net /MCU/SWCLK: track 42.8 -> 22.0 mm
- net /Input_driver/IN2: track 0.00 -> 20.3 mm
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- added copper zone on F.Cu, net +5VD
- added copper zone on F.Cu, net Net-(U901-FB)
- removed copper zone on B.Cu, net +12V
- removed copper zone on B.Cu, net +5VD
- removed copper zone on B.Cu, net /Battery_Module/BAT(+)
- removed copper zone on B.Cu, net Net-(D502-K)
- removed copper zone on B.Cu, net Net-(D503-A)
- removed copper zone on B.Cu, net Net-(U501-CSP)
- removed copper zone on B.Cu, net Net-(U901-FB)
Other:
- board size 74 x 108 mm -> 55 x 108 mm
- board text added: "01-1"
- board text added: "1-1"
- board text added: "230V AC"
- board text added: "AN-M1"
- board text added: "BAT+"
- board text added: "BAT-"
- board text added: "IN1"
- board text added: "IN2"
- board text added: "IN3"
- board text added: "IN4"
- board text added: "J1001"
- board text added: "O1-2"
- board text added: "O2-2"
- board text removed: "+"
- board text removed: "-"
- board text removed: "230VAC"
- board text removed: "3.7V 18650 Battery"
- board text removed: "M"
- board text removed: "SOLAR 12V"
- board text removed: "Universal Sensor RS485"
