File: govi_v3_Actuator_node_kicad.kicad_sch (KiCad schematic)
At the start: 5 parts

Commit message: "V1.0 final design"
Parts:
- removed H101, H102, H103, H104: MountingHole_Pad, MountingHole:MountingHole_3.2mm_M3_Pad_TopBottom, symbol Mechanical:MountingHole_Pad
Connections:
- no-connect marks 1 -> 0
Other:
- removed sheet MPPT_Charger_module
- sheet Input_driver ports: added INPUT2, INPUT3; removed none
- sheet MCU ports: added IN_2, IN_3; removed none
- note removed: "Mounting Holes M3"
